File: finalized-schematic/finalized-bluetooth-remote/finalized-bluetooth-remote.kicad_pcb (KiCad board)
At the start: 4 copper layers, 48 parts, among them J1 USB_C_Receptacle_USB2.0_16P, J2 Conn_01x02, Q1 DMG3415U, SW1 SW_Push, SW2 SW_Push, SW3 SW_Push, SW4 SW_Push, SW5 SW_SPDT, SW6 SW_Push, SW7 SW_Push, SW8 SW_SPDT, U1 MCP73831-2-OT, U2 MCP6001-OT, U3 AP2112K-3.3, U4 ESP32-S3-WROOM-1

Commit message: finished PCB design
Parts:
- added C11: 0.1uf, Capacitor_SMD:C_0603_1608Metric, F.Cu at (168.7, 102.5)
- added C12: 0.1uf, Capacitor_SMD:C_0603_1608Metric, F.Cu at (165.5, 104.5)
- added G***: LOGO, LOGO, F.Cu at (147.4, 77.6)
- added J3: Conn_02x05_Odd_Even, Connector_PinHeader_2.54mm:PinHeader_2x05_P2.54mm_Vertical, F.Cu at (133.2, 111.1)
- added R13: 1k, Resistor_SMD:R_0603_1608Metric, F.Cu at (167.9, 104.7)
- added TP1: TestPoint_Probe, TestPoint:TestPoint_Pad_D2.0mm, F.Cu at (135.1, 80.1)
- added TP2: TestPoint_Probe, TestPoint:TestPoint_Pad_D2.0mm, F.Cu at (186.8, 87.0)
- added TP3: TestPoint_Probe, TestPoint:TestPoint_Pad_D2.0mm, F.Cu at (178.1, 83.9)
- added TP4: TestPoint_Probe, TestPoint:TestPoint_Pad_D2.0mm, F.Cu at (149.0, 83.8)
- added TP5: TestPoint_Probe, TestPoint:TestPoint_Pad_D2.0mm, F.Cu at (138.6, 80.1)
- added kibuzzard-69D59D66: G***, kibuzzard-69D59D66, F.Cu at (181.6, 78.4)
- added kibuzzard-69D59D85: G***, kibuzzard-69D59D85, F.Cu at (178.2, 110.5)
- added kibuzzard-69D59DAB: G***, kibuzzard-69D59DAB, F.Cu at (187.7, 110.4)
- added kibuzzard-69D59DBA: G***, kibuzzard-69D59DBA, F.Cu at (148.2, 97.5)
- C10, C6: value 10uf -> 1uf; footprint Capacitor_SMD:C_0805_2012Metric -> Capacitor_SMD:C_0603_1608Metric
- C2: value 4.7uf -> 0.1uf; footprint Capacitor_SMD:C_0805_2012Metric -> Capacitor_SMD:C_0603_1608Metric
- C3: value 1uf -> 4.7uf; footprint Capacitor_SMD:C_0603_1608Metric -> Capacitor_SMD:C_0805_2012Metric
- C4: value 100uf -> 1uf; footprint Capacitor_Tantalum_SMD:CP_EIA-7343-31_Kemet-D -> Capacitor_SMD:C_0603_1608Metric
- C5: value 1uf -> 100uf; footprint Capacitor_SMD:C_0603_1608Metric -> Capacitor_Tantalum_SMD:CP_EIA-7343-31_Kemet-D
- C7: value 1uf -> 10uf; footprint Capacitor_SMD:C_0603_1608Metric -> Capacitor_SMD:C_0805_2012Metric
- C8: value 0.1uf -> 10uf; footprint Capacitor_SMD:C_0603_1608Metric -> Capacitor_SMD:C_0805_2012Metric
- H1, H2, H3, H4: value MountingHole_Pad -> MountingHole; footprint MountingHole:MountingHole_2.2mm_M2_Pad -> MountingHole:MountingHole_2.2mm_M2
- R8: value 33k -> 10k
- R9: value 10k -> 33k
- SW5: footprint Connector_PinHeader_2.54mm:PinHeader_1x02_P2.54mm_Vertical -> Connector_PinHeader_2.54mm:PinHeader_1x03_P2.54mm_Vertical
- SW6: value SW_Push -> SW_SPDT; footprint Button_Switch_SMD:SW_SPST_Omron_B3FS-100xP -> Connector_PinHeader_2.54mm:PinHeader_1x03_P2.54mm_Vertical
- SW7: footprint Button_Switch_SMD:SW_SPST_Omron_B3FS-100xP -> Button_Switch_SMD:SW_Push_1P1T_NO_CK_KMR2
- SW8: value SW_SPDT -> SW_Push; footprint Connector_PinHeader_2.54mm:PinHeader_1x03_P2.54mm_Vertical -> Button_Switch_SMD:SW_Push_1P1T_NO_CK_KMR2
- moved SW8 235.9 mm to (127.5, 109.5)
- moved J1 227.3 mm to (128.0, 87.2), turned to -90 degrees
- moved D1 224.9 mm to (142.6, 97.6), turned to 180 degrees
- moved C10 216.6 mm to (130.4, 101.9)
- moved C1 210.9 mm to (136.7, 103.3), turned to -90 degrees
- moved C2 207.9 mm to (139.2, 97.8)
- moved R11 207.1 mm to (130.5, 100.4), turned to 180 degrees
- moved R12 206.8 mm to (131.1, 107.5), turned to -90 degrees
- moved R3 206.1 mm to (127.5, 81.1), turned to 180 degrees
- moved U1 203.3 mm to (139.3, 100.6), turned to -90 degrees
- moved R2 203.0 mm to (130.5, 81.1)
- moved H3 200.1 mm to (125.8, 122.4)
- moved H1 199.0 mm to (125.8, 76.4)
- moved C6 198.0 mm to (148.9, 88.5)
- moved R7 197.8 mm to (135.9, 89.4), turned to 90 degrees
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Connections:
- C10 pad 1: +3.3V -> EN
- C3 pad 1: Net-(D5-K) -> +BATT
- C4 pad 1: +3.3V -> Net-(U3-VIN)
- C7 pad 1: EN -> +3.3V
- C8 pad 1: +BATT -> +3.3V
- R4 pad 1: Net-(D1-K) -> Net-(D3-K)
- R5 pad 1: Net-(D3-K) -> Net-(D1-K)
- R7 pad 1: +BATT -> GND
- R7 pad 2: Net-(U2-+) -> +5V
- R8 pad 1: Net-(U2-+) -> +BATT
- R8 pad 2: GND -> Net-(U2-+)
- R9 pad 1: GND -> Net-(U2-+)
- R9 pad 2: +5V -> GND
- SW6 pad 1: EN -> unconnected-(SW6-A-Pad1)
- SW6 pad 2: GND -> +BATT
- SW7 pad 1: BOOT -> EN
- SW8 pad 1: unconnected-(SW8-A-Pad1) -> BOOT
- SW8 pad 2: +BATT -> GND
- U4 pad 17: unconnected-(U4-IO9-Pad17) -> GPIO9
- U4 pad 18: unconnected-(U4-IO10-Pad18) -> GPIO10
- U4 pad 19: unconnected-(U4-IO11-Pad19) -> GPIO11
- U4 pad 20: unconnected-(U4-IO12-Pad20) -> GPIO12
- U4 pad 21: unconnected-(U4-IO13-Pad21) -> GPIO13
- U4 pad 22: unconnected-(U4-IO14-Pad22) -> GPIO14
- U4 pad 23: GPIO21 -> Net-(U4-IO21)
- U4 pad 8: unconnected-(U4-IO15-Pad8) -> GPIO15
- U4 pad 9: unconnected-(U4-IO16-Pad9) -> GPIO16
Routing:
- net +3.3V: track 0.00 -> 89.7 mm, vias 0 -> 2
- net BOOT: track 0.00 -> 87.9 mm, vias 0 -> 2
- net +BATT: track 0.00 -> 87.1 mm
- net GPIO16: track 0.00 -> 79.0 mm, vias 0 -> 1
- net GPIO5: track 0.00 -> 58.4 mm, vias 0 -> 2
- net GPIO14: track 0.00 -> 56.5 mm, vias 0 -> 1
- net GPIO1: track 0.00 -> 55.0 mm, vias 0 -> 2
- net GPIO15: track 0.00 -> 51.3 mm, vias 0 -> 1
- net +5V: track 0.00 -> 51.0 mm
- net GPIO4: track 0.00 -> 49.4 mm, vias 0 -> 2
- net GPIO2: track 0.00 -> 48.8 mm, vias 0 -> 2
- net EN: track 0.00 -> 47.2 mm, vias 0 -> 2
- net DATA+: track 0.00 -> 46.2 mm, vias 0 -> 2
- net GPIO6: track 0.00 -> 45.4 mm, vias 0 -> 2
- net GPIO7: track 0.00 -> 40.7 mm, vias 0 -> 2
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- added copper zone on B.Cu, net GND
- added copper zone on F.Cu, net GND
- added copper zone on In1.Cu, net GND
- added copper zone on In2.Cu, net GND
Other:
- board outline added: 70 x 50 mm
