File: finalized-schematic/finalized-bluetooth-remote/finalized-bluetooth-remote.kicad_sch (KiCad schematic)
At the start: 48 parts, among them J1 USB_C_Receptacle_USB2.0_16P, J2 Conn_01x02, Q1 DMG3415U, SW1 SW_Push, SW2 SW_Push, SW3 SW_Push, SW4 SW_Push, SW5 SW_SPDT, SW6 SW_Push, SW7 SW_Push, SW8 SW_SPDT, U1 MCP73831-2-OT, U2 MCP6001-OT, U3 AP2112K-3.3, U4 ESP32-S3-WROOM-1

Commit message: finished PCB design
Parts:
- removed H1, H2, H3, H4: MountingHole_Pad, MountingHole:MountingHole_2.2mm_M2_Pad, symbol Mechanical:MountingHole_Pad
- added C11, C12: 0.1uf, Capacitor_SMD:C_0603_1608Metric, symbol Device:C_US
- added H1, H2, H3, H4: MountingHole, MountingHole:MountingHole_2.2mm_M2, symbol Mechanical:MountingHole
- added J3: Conn_02x05_Odd_Even, Connector_PinHeader_2.54mm:PinHeader_2x05_P2.54mm_Vertical, symbol Connector_Generic:Conn_02x05_Odd_Even
- added R13: 1k, Resistor_SMD:R_0603_1608Metric, symbol Device:R_US
- added TP1, TP2, TP3, TP4, TP5: TestPoint_Probe, TestPoint:TestPoint_Pad_D2.0mm, symbol Connector:TestPoint_Probe
- SW5: footprint Connector_PinHeader_2.54mm:PinHeader_1x02_P2.54mm_Vertical -> Connector_PinHeader_2.54mm:PinHeader_1x03_P2.54mm_Vertical
- SW7: renamed from SW6; footprint Button_Switch_SMD:SW_SPST_Omron_B3FS-100xP -> Button_Switch_SMD:SW_Push_1P1T_NO_CK_KMR2
- SW8: renamed from SW7; footprint Button_Switch_SMD:SW_SPST_Omron_B3FS-100xP -> Button_Switch_SMD:SW_Push_1P1T_NO_CK_KMR2
- renumbered C7 to C10, C8 to C2, C2 to C3, C3 to C4, C4 to C5, C5 to C6, C6 to C7, C10 to C8, R5 to R4, R4 to R5, R9 to R7, R7 to R8, R8 to R9, SW8 to SW6
Connections:
- net +3.3V: now also C12.1, J3.1 (Pin_1), TP4.1
- net +5V: now also TP1.1
- net +BATT: now also TP2.1
- net GND: now also C11.2, C12.2, J3.3 (Pin_3), TP3.1
- net GPIO21: now also R13.1; no longer U4.23 (IO21)
- net at D5.1 (K), F1.1, Q1.1 (D)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: no longer C4.1
- net at F1.2, U3.1 (VIN): now also C4.1, TP5.1
- net GPIO9: now reaches U4.17 (IO9)
- net GPIO9: now also J3.5 (Pin_5)
- net GPIO10: now reaches U4.18 (IO10)
- net GPIO10: now also J3.7 (Pin_7)
- net GPIO11: now reaches U4.19 (IO11)
- net GPIO11: now also J3.9 (Pin_9)
- net GPIO12: now reaches U4.20 (IO12)
- net GPIO12: now also J3.2 (Pin_2)
- net GPIO13: now reaches U4.21 (IO13)
- net GPIO13: now also J3.4 (Pin_4)
- net GPIO14: now reaches U4.22 (IO14)
- net GPIO14: now also J3.6 (Pin_6)
- net GPIO15: now reaches U4.8 (IO15)
- net GPIO15: now also J3.8 (Pin_8)
- net GPIO16: now reaches U4.9 (IO16)
- net GPIO16: now also J3.10 (Pin_10)
- new net: C11.1, R13.2, U4.23 (IO21)
- no-connect marks 29 -> 21
Other:
- note added: "Avoid GPIO: * GPIO0 * GPIO3 * GPIO35-37 * GPIO39-42 * GPIO43-44 * GPIO45-46"
- note added: "External Header"
- note added: "For a 500 mAh LiPo battery (the battery also needs built-in protection circuitry)"
- note added: "For future proofing"
- note added: "Net Test Points"
- note removed: "* SW1 - Play/pause and accept/decline/end call | Volume up * SW2 - Previous song | Volume down * SW3 - Next song | Mute volume * SW4 - Change control set"
- note removed: "Avoid GPIO: * GPIO3 * GPIO35 * GPIO36 * GPIO37 * GPIO45 * GPIO46"
- note removed: "For a 400 mAh LiPo battery (the battery also needs built-in protection circuitry)"
- moved on the sheet: C1, C10, C2, C3, C4, C5, C6, C7, C8, C9, D1, D2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
