File: finalized-schematic (expensive)/finalized-bluetooth-remote/finalized-bluetooth-remote.kicad_pcb (KiCad board)
At the start: 4 copper layers, 70 x 50 mm, 62 parts, among them J1 USB_C_Receptacle_USB2.0_16P, J2 Conn_01x02, J3 Conn_02x05_Odd_Even, Q1 DMG3415U, SW1 SW_Push, SW2 SW_Push, SW3 SW_Push, SW4 SW_Push, SW5 SW_SPDT, SW6 SW_SPDT, SW7 SW_Push, SW8 SW_Push, U1 MCP73831-2-OT, U2 MCP6001-OT, U3 AP2112K-3.3, U4 ESP32-S3-WROOM-1

Commit message: finished version of finalized schematic
Parts:
- moved J2 0.28 mm to (188.5, 96.6), turned to -90 degrees
Routing:
- net Net-(J2-Pin_2): track 8.36 -> 11.3 mm
- removed copper zone on In2.Cu, net GND
Changed lines of the file:
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@@
 			(outputformat 1)
 			(mirror no)
-			(drillshape 1)
+			(drillshape 0)
 			(scaleselection 1)
-			(outputdirectory "")
+			(outputdirectory "../../../")
 		)
 	)
@@
 	(footprint "Connector_JST:JST_PH_S2B-PH-SM4-TB_1x02-1MP_P2.00mm_Horizontal"
 		(layer "F.Cu")
-		(at 188.228 96.496 90)
+		(at 188.468 96.647 -90)
 		(descr "JST PH series connector, S2B-PH-SM4-TB (http://www.jst-mfg.com/product/pdf/eng/ePH.pdf), generated with kicad-footprint-generator")
 		(tags "connector JST PH horizontal")
 		(property "Reference" "J2"
-			(at 0 -5.8 90)
+			(at -0.127 5.969 180)
 			(layer "F.SilkS")
 			(effects
@@
 		(attr smd)
 		(fp_line
-			(start 4.06 -3.31)
-			(end 3.04 -3.31)
+			(start -2.34 4.51)
+			(end 2.34 4.51)
 			(stroke
 				(width 0.12)
@@
 		)
 		(fp_line
-			(start 3.04 -3.31)
-			(end 3.04 -1.71)
+			(start -4.06 0.94)
+			(end -4.06 -3.31)
 			(stroke
 				(width 0.12)
@@
 		)
 		(fp_line
-			(start -3.04 -3.31)
-			(end -3.04 -1.71)
+			(start 4.06 0.94)
+			(end 4.06 -3.31)
 			(stroke
 				(width 0.12)
@@
 		)
 		(fp_line
-			(start -4.06 -3.31)
-			(end -3.04 -3.31)
+			(start -3.04 -1.71)
+			(end -1.76 -1.71)
 			(stroke
 				(width 0.12)
@@
 		)
 		(fp_line
-			(start 3.04 -1.71)
-			(end 1.76 -1.71)
+			(start -1.76 -1.71)
+			(end -1.76 -4.6)
 			(stroke
 				(width 0.12)
@@
 		)
 		(fp_line
-			(start -1.76 -1.71)
-			(end -1.76 -4.6)
+			(start 3.04 -1.71)
+			(end 1.76 -1.71)
 			(stroke
 				(width 0.12)
@@
 		)
 		(fp_line
-			(start -3.04 -1.71)
-			(end -1.76 -1.71)
+			(start -4.06 -3.31)
+			(end -3.04 -3.31)
 			(stroke
 				(width 0.12)
@@
 		)
 		(fp_line
-			(start 4.06 0.94)
-			(end 4.06 -3.31)
+			(start -3.04 -3.31)
+			(end -3.04 -1.71)
 			(stroke
 				(width 0.12)
@@
 		)
 		(fp_line
-			(start -4.06 0.94)
-			(end -4.06 -3.31)
+			(start 3.04 -3.31)
+			(end 3.04 -1.71)
 			(stroke
 				(width 0.12)
@@
 		)
 		(fp_line
-			(start -2.34 4.51)
-			(end 2.34 4.51)
+			(start 4.06 -3.31)
+			(end 3.04 -3.31)
 			(stroke
 				(width 0.12)
@@
 		)
 		(fp_line
-			(start 2 -5.1)
-			(end 2 -3.7)
+			(start -4.6 5.1)
+			(end -4.6 0.69)
 			(stroke
 				(width 0.05)
@@
 		)
 		(fp_line
-			(start -2 -5.1)
-			(end 2 -5.1)
+			(start -2.1 5.1)
+			(end -4.6 5.1)
 			(stroke
 				(width 0.05)
@@
 		)
 		(fp_line
-			(start 4.45 -3.7)
-			(end 4.45 0.69)
+			(start 2.1 5.1)
+			(end 2.1 4.9)
 			(stroke
 				(width 0.05)
@@
 		)
 		(fp_line
-			(start 2 -3.7)
-			(end 4.45 -3.7)
+			(start 4.6 5.1)
+			(end 2.1 5.1)
 			(stroke
 				(width 0.05)
@@
 		)
 		(fp_line
-			(start -2 -3.7)
-			(end -2 -5.1)
+			(start -2.1 4.9)
+			(end -2.1 5.1)
 			(stroke
 				(width 0.05)
@@
 		)
 		(fp_line
-			(start -4.45 -3.7)
-			(end -2 -3.7)
+			(start 2.1 4.9)
+			(end -2.1 4.9)
 			(stroke
 				(width 0.05)
@@
 		)
 		(fp_line
-			(start 4.6 0.69)
-			(end 4.6 5.1)
+			(start -4.6 0.69)
+			(end -4.45 0.69)
 			(stroke
 				(width 0.05)
@@
 		)
 		(fp_line
-			(start 4.45 0.69)
-			(end 4.6 0.69)
+			(start -4.45 0.69)
+			(end -4.45 -3.7)
 			(stroke
 				(width 0.05)
@@
 		)
 		(fp_line
-			(start -4.45 0.69)
-			(end -4.45 -3.7)
+			(start 4.45 0.69)
+			(end 4.6 0.69)
 			(stroke
 				(width 0.05)
@@
 		)
 		(fp_line
-			(start -4.6 0.69)
-			(end -4.45 0.69)
+			(start 4.6 0.69)
+			(end 4.6 5.1)
 			(stroke
 				(width 0.05)
@@
 		)
 		(fp_line
-			(start 2.1 4.9)
-			(end -2.1 4.9)
+			(start -4.45 -3.7)
+			(end -2 -3.7)
 			(stroke
 				(width 0.05)
@@
 		)
 		(fp_line
-			(start -2.1 4.9)
-			(end -2.1 5.1)
+			(start -2 -3.7)
+			(end -2 -5.1)
 			(stroke
 				(width 0.05)
@@
 		)
 		(fp_line
-			(start 4.6 5.1)
-			(end 2.1 5.1)
+			(start 2 -3.7)
+			(end 4.45 -3.7)
 			(stroke
 				(width 0.05)
@@
 		)
 		(fp_line
-			(start 2.1 5.1)
-			(end 2.1 4.9)
+			(start 4.45 -3.7)
+			(end 4.45 0.69)
 			(stroke
 				(width 0.05)
@@
 		)
 		(fp_line
-			(start -2.1 5.1)
-			(end -4.6 5.1)
+			(start -2 -5.1)
+			(end 2 -5.1)
 			(stroke
 				(width 0.05)
@@
 		)
 		(fp_line
-			(start -4.6 5.1)
-			(end -4.6 0.69)
+			(start 2 -5.1)
+			(end 2 -3.7)
 			(stroke
 				(width 0.05)
@@
 		)
 		(fp_line
-			(start 3.95 -3.2)
+			(start -3.95 4.4)
 			(end 3.95 4.4)
 			(stroke
@@
 		)
 		(fp_line
-			(start 3.15 -3.2)
-			(end 3.95 -3.2)
+			(start -1 -0.892893)
+			(end -0.5 -1.6)
 			(stroke
 				(width 0.1)
@@
 		)
 		(fp_line
-			(start -3.15 -3.2)
-			(end -3.15 -1.6)
+			(start -3.15 -1.6)
+			(end 3.15 -1.6)
 			(stroke
 				(width 0.1)
@@
 		)
 		(fp_line
-			(start -3.95 -3.2)
-			(end -3.15 -3.2)
+			(start -1.5 -1.6)
+			(end -1 -0.892893)
 			(stroke
 				(width 0.1)
@@
 		)
 		(fp_line
-			(start -3.95 -3.2)
-			(end -3.95 4.4)
+			(start 3.15 -1.6)
+			(end 3.15 -3.2)
 			(stroke
 				(width 0.1)
@@
 		)
 		(fp_line
-			(start 3.15 -1.6)
-			(end 3.15 -3.2)
+			(start -3.95 -3.2)
+			(end -3.95 4.4)
 			(stroke
 				(width 0.1)
@@
 		)
 		(fp_line
-			(start -1.5 -1.6)
-			(end -1 -0.892893)
+			(start -3.95 -3.2)
+			(end -3.15 -3.2)
 			(stroke
 				(width 0.1)
@@
 		)
 		(fp_line
-			(start -3.15 -1.6)
-			(end 3.15 -1.6)
+			(start -3.15 -3.2)
+			(end -3.15 -1.6)
 			(stroke
 				(width 0.1)
@@
 		)
 		(fp_line
-			(start -1 -0.892893)
-			(end -0.5 -1.6)
+			(start 3.15 -3.2)
+			(end 3.95 -3.2)
 			(stroke
 				(width 0.1)
@@
 		)
 		(fp_line
-			(start -3.95 4.4)
+			(start 3.95 -3.2)
 			(end 3.95 4.4)
 			(stroke
@@
 		)
 		(pad "1" smd roundrect
-			(at -1 -2.85 90)
+			(at -1 -2.85 270)
 			(size 1 3.5)
 			(layers "F.Cu" "F.Mask" "F.Paste")
@@
 		)
 		(pad "2" smd roundrect
-			(at 1 -2.85 90)
+			(at 1 -2.85 270)
 			(size 1 3.5)
 			(layers "F.Cu" "F.Mask" "F.Paste")
@@
 		)
 		(pad "MP" smd roundrect
-			(at -3.35 2.9 90)
+			(at -3.35 2.9 270)
 			(size 1.5 3.4)
 			(layers "F.Cu" "F.Mask" "F.Paste")
@@
 		)
 		(pad "MP" smd roundrect
-			(at 3.35 2.9 90)
+			(at 3.35 2.9 270)
 			(size 1.5 3.4)
 			(layers "F.Cu" "F.Mask" "F.Paste")
@@
 	)
 	(via
-		(at 186.196 91.162)
+		(at 192.659 93.98)
 		(size 0.8)
 		(drill 0.4)
@@
 	)
 	(via
-		(at 184.291 99.036)
+		(at 187.706 102.87)
 		(size 0.8)
 		(drill 0.4)
@@
 	)
 	(segment
-		(start 191.123 89.511)
-		(end 185.378 95.256)
+		(start 191.318 97.647)
+		(end 189.976 97.647)
+		(width 0.64)
+		(layer "F.Cu")
+		(net 21)
+	)
+	(segment
+		(start 189.976 97.647)
+		(end 188.341 96.012)
+		(width 0.64)
+		(layer "F.Cu")
+		(net 21)
+	)
+	(segment
+		(start 188.341 92.293)
+		(end 191.123 89.511)
 		(width 0.64)
 		(layer "F.Cu")
@@
 	)
 	(segment
-		(start 185.378 95.256)
-		(end 185.378 95.496)
+		(start 188.341 96.012)
+		(end 188.341 92.293)
 		(width 0.64)
 		(layer "F.Cu")
@@
 		(net 1)
 		(net_name "GND")
-		(layers "F.Cu" "B.Cu" "In1.Cu" "In2.Cu")
+		(layers "F.Cu" "B.Cu" "In1.Cu")
 		(hatch edge 0.5)
 		(connect_pads
