File: finalized-schematic (expensive)/finalized-bluetooth-remote/finalized-bluetooth-remote.kicad_sch (KiCad schematic)
At the start: 57 parts, among them J1 USB_C_Receptacle_USB2.0_16P, J2 Conn_01x02, J3 Conn_02x05_Odd_Even, Q1 DMG3415U, SW1 SW_Push, SW2 SW_Push, SW3 SW_Push, SW4 SW_Push, SW5 SW_SPDT, SW6 SW_SPDT, SW7 SW_Push, SW8 SW_Push, U1 MCP73831-2-OT, U2 MCP6001-OT, U3 AP2112K-3.3, U4 ESP32-S3-WROOM-1

Commit message: finished version of finalized schematic
Parts:
- C1, C3: LCSC (none) -> C1746
- C10, C4, C6: LCSC (none) -> C1592
- C11, C12, C2, C9: LCSC (none) -> C1590
- C5: LCSC (none) -> C90975
- C7, C8: LCSC (none) -> C1713
- D1, D3, D4: LCSC (none) -> C2288
- D2: LCSC (none) -> C2827688
- D5: LCSC (none) -> C77337
- D6: LCSC (none) -> C283866
- F1: LCSC (none) -> C12558
- J1: LCSC (none) -> C165948
- J2: LCSC (none) -> C295747
- J3, SW5, SW6, TP1, TP2, TP3, TP4, TP5: now left out of the parts list
- Q1: LCSC (none) -> C7202986
- R1, R11, R2, R3: LCSC (none) -> C177348
- R10, R12, R7, R8: LCSC (none) -> C177337
- R13, R4, R5, R6: LCSC (none) -> C177343
- R9: LCSC (none) -> C177291
- SW1, SW2, SW3, SW4: LCSC (none) -> C87038
- SW7, SW8: LCSC (none) -> C72443
- U1: LCSC (none) -> C14879
- U2: LCSC (none) -> C21403
- U3: LCSC (none) -> C22365427
- U4: LCSC (none) -> C2913199
