File: Schematics/finalized-schematic (V3)/finalized-bluetooth-remote/finalized-bluetooth-remote.kicad_pcb (KiCad board)
At the start: 4 copper layers, 70 x 50 mm, 35 parts, among them J1 Conn_01x02, SW1 SW_SPDT, SW2 SW_Push, SW3 SW_Push, SW4 SW_Push, SW5 SW_Push, SW6 SW_SPDT, U1 XIAO ESP32C3, U2 OPA340P

Commit message: Confirm PCB V3
Parts:
- moved J1 1.80 mm to (178.3, 92.2), turned to 90 degrees
Routing:
- net -BATT: track 78.0 -> 72.0 mm, vias 2 -> 1
- net Net-(J1-Pin_2): track 12.4 -> 9.98 mm
